File: PCB/_saved_Microcontroller.sch (KiCad schematic (older format))
At the start: 19 parts, among them U8 ATSAM4S, Y1 12MHz .25%

Commit message: Generated BOM, fixed component names in schematic
Changed component names on output resistors and status LED to match that
in PCB
Parts:
- gave numbers to parts that had none: 1
- renumbered D1 to Status1
Changed lines of the file:
@@
 $EndComp
 $Comp
-L Led_Small D1
+L Led_Small Status1
 U 1 1 56BC8E49
 P 5550 6750
-F 0 "D1" H 5500 6875 50  0000 L CNN
+F 0 "Status1" H 5500 6875 50  0000 L CNN
 F 1 "Led_Small" H 5375 6650 50  0000 L CNN
 F 2 "LEDs:LED_0603" V 5550 6750 50  0001 C CNN
@@
 Erase pins, short these to erase program then reset
 $Comp
-L CONN_01X02 P?
+L CONN_01X02 P3
 U 1 1 570CE395
 P 1150 7000
-F 0 "P?" H 1150 7150 50  0000 C CNN
+F 0 "P3" H 1150 7150 50  0000 C CNN
 F 1 "CONN_01X02" V 1250 7000 50  0000 C CNN
 F 2 "" H 1150 7000 50  0000 C CNN
